File: WPC-S Battery Board.kicad_pcb (KiCad board)
At the start: 2 copper layers, 54 x 123 mm, 8 parts, among them J101 Conn_01x05

Commit message: Specify JLC order number location
Other:
- board text added: "JLCJLCJLCJLC"
Changed lines of the file:
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@@
   (gr_line (start 91.35 159.68) (end 91.35 42.18)
     (stroke (width 0.1) (type default)) (layer "Edge.Cuts"))
+  (gr_text "JLCJLCJLCJLC" (at 123.617858 71.57175) (layer "B.SilkS")
+    (effects (font (size 1 1) (thickness 0.15)) (justify left bottom mirror))
+  )
   (gr_text "bdash's battery board\nWPC-S ${VERSION}" (at 118.04 55.3) (layer "F.SilkS")
     (effects (font (face "Menlo") (size 1.25 1.25) (thickness 0.2) bold) (justify bottom))
